Commit message: first robot model finish stabel

File: models/robot_6_joint.urdf.xacro (robot description, xacro)
@@ -1,4 +1,5 @@
 <?xml version="1.0"?>
 <robot xmlns:xacro="http://www.ros.org/wiki/xacro"  name="robot">
+<xacro:include filename="materials.xacro" />
     <!-- base link-->
     <link name="base_link">
@@ -6,4 +7,5 @@
     <!--main base link-->
     <xacro:include filename="robot_base_square.xacro" />
+    <!-- base to chasiis-->
     <joint name="base_link_joint" type="fixed">
         <parent link="base_link"/>
@@ -11,3 +13,28 @@
         <origin xyz="-0.21 0 0"/>
     </joint>
+    <xacro:include filename="robot_legs.xacro" />
+    <!-- base to leg 1-->
+    <joint name="base_leg1_joint" type="revolute">
+        <parent link="main_base_square"/>
+        <child link="leg1_1"/>
+        <origin xyz="0.46 0 0" rpy="-${pi/2} 0 0"/>
+        <limit lower="0" upper="3.14" effort="10" velocity="3"/>
+        <axis xyz="0 0 1"/>
+    </joint>
+        <!-- base to leg 2-->
+    <joint name="base_leg2_joint" type="revolute">
+        <parent link="main_base_square"/>
+        <child link="leg2_1"/>
+        <origin xyz="0 0.225 0" rpy="-${pi/2} 0 0"/>
+        <limit lower="0" upper="3.14" effort="10" velocity="3"/>
+        <axis xyz="0 0 1"/>
+    </joint>
+        <!-- base to leg 3-->
+    <joint name="base_leg3_joint" type="revolute">
+        <parent link="main_base_square"/>
+        <child link="leg3_1"/>
+        <origin xyz="0 -0.225 0" rpy="${pi/2} 0 0"/>
+        <limit lower="0" upper="3.14" effort="10" velocity="3"/>
+        <axis xyz="0 0 -1"/>
+    </joint>
 </robot>

File: models/robot_base_square.xacro (robot description, xacro)
@@ -1,5 +1,4 @@
 <?xml version="1.0"?>
 <robot xmlns:xacro="http://www.ros.org/wiki/xacro" >
-<xacro:include filename="materials.xacro" />
 <link name="main_base_square">
     <visual>

Commit message: robot_with_inertial_tags

File: models/robot_6_joint.urdf.xacro (robot description, xacro)
@@ -2,4 +2,5 @@
 <robot xmlns:xacro="http://www.ros.org/wiki/xacro"  name="robot">
 <xacro:include filename="materials.xacro" />
+<xacro:include filename="inertial_macros.xacro" />
     <!-- base link-->
     <link name="base_link">

File: models/robot_base_square.xacro (robot description, xacro)
@@ -9,4 +9,13 @@
         <material name="magenta"/>
     </visual>
+    <collision>
+        <origin xyz="0.21 0 0"/>
+        <geometry>
+            <box size="0.5 0.4 0.1"/>
+        </geometry>
+    </collision>
+    <xacro:inertial_box mass="2" x="0.5" y="0.4" z="0.1">
+       <origin xyz="0.21 0 0" rpy="0 0 0"/>
+    </xacro:inertial_box>
 </link>
 </robot>

File: models/robot_legs.xacro (robot description, xacro)
@@ -10,4 +10,13 @@
         <material name="orange"/>
     </visual>
+    <collision>
+        <origin xyz="0.15 0 0"/>
+        <geometry>
+            <box size="0.3 0.08 0.05"/>
+        </geometry>
+    </collision>
+    <xacro:inertial_box mass="0.3" x="0.3" y="0.08" z="0.05">
+       <origin xyz="0.15 0 0" rpy="0 0 0"/>
+    </xacro:inertial_box>
 </link>
 <joint name="leg1_joint" type="revolute">
@@ -26,4 +35,13 @@
         <material name="yellow"/>
     </visual>
+    <collision>
+        <origin xyz="0.25 0 0"/>
+        <geometry>
+            <box size="0.5 0.08 0.05"/>
+        </geometry>
+    </collision>
+    <xacro:inertial_box mass="0.5" x="0.5" y="0.08" z="0.05">
+       <origin xyz="0.25 0 0" rpy="0 0 0"/>
+    </xacro:inertial_box>
 </link>
 <!-- leg 2-->
@@ -36,4 +54,13 @@
         <material name="orange"/>
     </visual>
+    <collision>
+        <origin xyz="0.15 0 0"/>
+        <geometry>
+            <box size="0.3 0.08 0.05"/>
+        </geometry>
+    </collision>
+    <xacro:inertial_box mass="0.3" x="0.3" y="0.08" z="0.05">
+       <origin xyz="0.15 0 0" rpy="0 0 0"/>
+    </xacro:inertial_box>
 </link>
 <joint name="leg2_joint" type="revolute">
@@ -52,4 +79,13 @@
         <material name="yellow"/>
     </visual>
+    <collision>
+        <origin xyz="0.25 0 0"/>
+        <geometry>
+            <box size="0.5 0.08 0.05"/>
+        </geometry>
+    </collision>
+    <xacro:inertial_box mass="0.5" x="0.5" y="0.08" z="0.05">
+       <origin xyz="0.25 0 0" rpy="0 0 0"/>
+    </xacro:inertial_box>
 </link>
 <!-- leg 3-->
@@ -62,4 +98,13 @@
         <material name="orange"/>
     </visual>
+    <collision>
+        <origin xyz="0.15 0 0"/>
+        <geometry>
+            <box size="0.3 0.08 0.05"/>
+        </geometry>
+    </collision>
+    <xacro:inertial_box mass="0.3" x="0.3" y="0.08" z="0.05">
+       <origin xyz="0.15 0 0" rpy="0 0 0"/>
+    </xacro:inertial_box>
 </link>
 <joint name="leg3_joint" type="revolute">
@@ -78,4 +123,13 @@
         <material name="yellow"/>
     </visual>
+    <collision>
+        <origin xyz="0.25 0 0"/>
+        <geometry>
+            <box size="0.5 0.08 0.05"/>
+        </geometry>
+    </collision>
+    <xacro:inertial_box mass="0.5" x="0.5" y="0.08" z="0.05">
+       <origin xyz="0.25 0 0" rpy="0 0 0"/>
+    </xacro:inertial_box>
 </link>
 </robot>
