Commit message: robot_final

File: models/robot_base_square.xacro (robot description, xacro)
@@ -1,4 +1,5 @@
 <?xml version="1.0"?>
 <robot xmlns:xacro="http://www.ros.org/wiki/xacro" >
+<!--main base plate-->
 <link name="main_base_square">
     <visual>
@@ -7,5 +8,5 @@
             <box size="0.5 0.4 0.1"/>
         </geometry>
-        <material name="magenta"/>
+        <material name="white"/>
     </visual>
     <collision>
@@ -19,3 +20,34 @@
     </xacro:inertial_box>
 </link>
+<gazebo reference="main_base_square">
+    <material>Gazebo/White</material>
+</gazebo>
+<!--joint between base plate and lidar-->
+<joint name="base_lidar_joint" type="fixed">
+    <parent link="main_base_square"/>
+    <child link="lidar"/>
+    <origin xyz="0.21 0 0.05" rpy="0 0 0"/>
+</joint>
+<!--lidar link-->
+<link name="lidar">
+    <visual>
+        <origin xyz="0 0 0.025"/>
+        <geometry>
+            <cylinder length="0.04" radius="0.05"/>
+        </geometry>
+        <material name="black"/>
+    </visual>
+    <collision>
+        <origin xyz="0 0 0.025"/>
+        <geometry>
+            <cylinder length="0.04" radius="0.05"/>
+        </geometry>
+    </collision>
+    <xacro:inertial_cylinder mass="2" length="0.04" radius="0.05">
+       <origin xyz="0 0 0.025" rpy="0 0 0"/>
+    </xacro:inertial_cylinder>
+</link>
+<gazebo reference="lidar">
+    <material>Gazebo/Black</material>
+</gazebo>
 </robot>

File: models/robot_legs.xacro (robot description, xacro)
@@ -20,4 +20,7 @@
     </xacro:inertial_box>
 </link>
+<gazebo reference="leg1_1">
+    <material>Gazebo/Orange</material>
+</gazebo>
 <joint name="leg1_joint" type="revolute">
     <parent link="leg1_1"/>
@@ -45,4 +48,7 @@
     </xacro:inertial_box>
 </link>
+<gazebo reference="leg1_2">
+    <material>Gazebo/Yellow</material>
+</gazebo>
 <!-- leg 2-->
 <link name="leg2_1">
@@ -64,4 +70,7 @@
     </xacro:inertial_box>
 </link>
+<gazebo reference="leg2_1">
+    <material>Gazebo/Orange</material>
+</gazebo>
 <joint name="leg2_joint" type="revolute">
     <parent link="leg2_1"/>
@@ -89,4 +98,7 @@
     </xacro:inertial_box>
 </link>
+<gazebo reference="leg2_2">
+    <material>Gazebo/Yellow</material>
+</gazebo>
 <!-- leg 3-->
 <link name="leg3_1">
@@ -108,4 +120,7 @@
     </xacro:inertial_box>
 </link>
+<gazebo reference="leg3_1">
+    <material>Gazebo/Orange</material>
+</gazebo>
 <joint name="leg3_joint" type="revolute">
     <parent link="leg3_1"/>
@@ -133,3 +148,6 @@
     </xacro:inertial_box>
 </link>
+<gazebo reference="leg3_2">
+    <material>Gazebo/Yellow</material>
+</gazebo>
 </robot>
