Commit message: robot_control_working_from_enviorment

File: models/robot_6_joint/robot_legs.xacro (robot description, xacro)
@@ -131,5 +131,5 @@
     <limit lower="-1.57" upper="1.57" effort="200.0" velocity="4"/>
     <dynamics friction="0.0" />
-    <axis xyz="0 0 1"/>
+    <axis xyz="0 0 -1"/>
 </joint>
 <link name="leg3_2">
