Commit message: robot moving with command

File: models/robot_6_joint/robot_6_joint.urdf.xacro (robot description, xacro)
@@ -20,5 +20,6 @@
         <child link="leg1_1"/>
         <origin xyz="0.46 0 0" rpy="-${pi/2} 0 0"/>
-        <limit lower="0" upper="3.14" effort="10" velocity="3"/>
+        <limit lower="0" upper="3.14" effort="200.0" velocity="4.0"/>
+        <dynamics friction="0.0" />
         <axis xyz="0 0 1"/>
     </joint>
@@ -28,5 +29,6 @@
         <child link="leg2_1"/>
         <origin xyz="0 0.225 0" rpy="-${pi/2} 0 0"/>
-        <limit lower="0" upper="3.14" effort="10" velocity="3"/>
+        <limit lower="0" upper="3.14" effort="200.0" velocity="4.0"/>
+        <dynamics friction="0.0" />
         <axis xyz="0 0 1"/>
     </joint>
@@ -36,5 +38,6 @@
         <child link="leg3_1"/>
         <origin xyz="0 -0.225 0" rpy="${pi/2} 0 0"/>
-        <limit lower="0" upper="3.14" effort="10" velocity="3"/>
+        <limit lower="0" upper="3.14" effort="200.0" velocity="4.0"/>
+        <dynamics friction="0.0" />
         <axis xyz="0 0 -1"/>
     </joint>

File: models/robot_6_joint/robot_base_square.xacro (robot description, xacro)
@@ -16,5 +16,5 @@
         </geometry>
     </collision>
-    <xacro:inertial_box mass="2" x="0.5" y="0.4" z="0.1">
+    <xacro:inertial_box mass="1" x="0.5" y="0.4" z="0.1">
        <origin xyz="0.21 0 0" rpy="0 0 0"/>
     </xacro:inertial_box>
@@ -44,5 +44,5 @@
         </geometry>
     </collision>
-    <xacro:inertial_cylinder mass="2" length="0.04" radius="0.05">
+    <xacro:inertial_cylinder mass="0.1" length="0.04" radius="0.05">
        <origin xyz="0 0 0.025" rpy="0 0 0"/>
     </xacro:inertial_cylinder>

File: models/robot_6_joint/robot_legs.xacro (robot description, xacro)
@@ -27,5 +27,6 @@
     <child link="leg1_2"/>
     <origin xyz="0.3 0 0"/>
-    <limit lower="-1.57" upper="1.57" effort="100" velocity="3"/>
+    <limit lower="-1.57" upper="1.57" effort="200.0" velocity="4.0"/>
+    <dynamics friction="0.0" />
     <axis xyz="0 0 1"/>
 </joint>
@@ -77,5 +78,6 @@
     <child link="leg2_2"/>
     <origin xyz="0.3 0 0"/>
-    <limit lower="-1.57" upper="1.57" effort="100" velocity="3"/>
+    <limit lower="-1.57" upper="1.57" effort="200.0" velocity="4.0"/>
+    <dynamics friction="0.0" />
     <axis xyz="0 0 1"/>
 </joint>
@@ -127,5 +129,6 @@
     <child link="leg3_2"/>
     <origin xyz="0.3 0 0"/>
-    <limit lower="-1.57" upper="1.57" effort="100" velocity="3"/>
+    <limit lower="-1.57" upper="1.57" effort="200.0" velocity="4"/>
+    <dynamics friction="0.0" />
     <axis xyz="0 0 1"/>
 </joint>

File: models/robot_6_joint/robot_transmission.xacro (robot description, xacro)
@@ -42,5 +42,5 @@
     <actuator name="leg1_joint_motor">
         <hardwareInterface>hardware_interface/EffortJointInterface</hardwareInterface>
-        <mechanicalReduction>1</mechanicalReduction>
+        <mechanicalReduction>100</mechanicalReduction>
     </actuator>
 </transmission>
@@ -53,5 +53,5 @@
     <actuator name="leg2_joint_motor">
         <hardwareInterface>hardware_interface/EffortJointInterface</hardwareInterface>
-        <mechanicalReduction>1</mechanicalReduction>
+        <mechanicalReduction>100</mechanicalReduction>
     </actuator>
 </transmission>
@@ -64,5 +64,5 @@
     <actuator name="leg3_joint_motor">
         <hardwareInterface>hardware_interface/EffortJointInterface</hardwareInterface>
-        <mechanicalReduction>1</mechanicalReduction>
+        <mechanicalReduction>100</mechanicalReduction>
     </actuator>
 </transmission>
@@ -72,4 +72,6 @@
         <robotNamespace>/robot_6_joint</robotNamespace>
         <robotSimType>gazebo_ros_control/DefaultRobotHWSim</robotSimType>
+        <updateRate>60.0</updateRate>
+        <alwaysOn>true</alwaysOn>
     </plugin>
 </gazebo>

Commit message: working

File: models/robot_6_joint/robot_6_joint.urdf.xacro (robot description, xacro)
@@ -20,5 +20,5 @@
         <child link="leg1_1"/>
         <origin xyz="0.46 0 0" rpy="-${pi/2} 0 0"/>
-        <limit lower="0" upper="3.14" effort="200.0" velocity="4.0"/>
+        <limit lower="1" upper="2" effort="200.0" velocity="4.0"/>
         <dynamics friction="0.0" />
         <axis xyz="0 0 1"/>
@@ -29,5 +29,5 @@
         <child link="leg2_1"/>
         <origin xyz="0 0.225 0" rpy="-${pi/2} 0 0"/>
-        <limit lower="0" upper="3.14" effort="200.0" velocity="4.0"/>
+        <limit lower="1" upper="2" effort="200.0" velocity="4.0"/>
         <dynamics friction="0.0" />
         <axis xyz="0 0 1"/>
@@ -38,5 +38,5 @@
         <child link="leg3_1"/>
         <origin xyz="0 -0.225 0" rpy="${pi/2} 0 0"/>
-        <limit lower="0" upper="3.14" effort="200.0" velocity="4.0"/>
+        <limit lower="1" upper="2" effort="200.0" velocity="4.0"/>
         <dynamics friction="0.0" />
         <axis xyz="0 0 -1"/>

File: models/robot_6_joint/robot_base_square.xacro (robot description, xacro)
@@ -16,5 +16,5 @@
         </geometry>
     </collision>
-    <xacro:inertial_box mass="8" x="0.5" y="0.4" z="0.1">
+    <xacro:inertial_box mass="5" x="0.5" y="0.4" z="0.1">
        <origin xyz="0.21 0 0" rpy="0 0 0"/>
     </xacro:inertial_box>

File: models/robot_6_joint/robot_legs.xacro (robot description, xacro)
@@ -29,5 +29,5 @@
     <child link="leg1_2"/>
     <origin xyz="0.3 0 0"/>
-    <limit lower="-1.57" upper="1.57" effort="200.0" velocity="4.0"/>
+    <limit lower="0" upper="1" effort="200.0" velocity="4.0"/>
     <dynamics friction="0.0" />
     <axis xyz="0 0 1"/>
@@ -130,5 +130,5 @@
     <child link="leg2_2"/>
     <origin xyz="0.3 0 0"/>
-    <limit lower="-1.57" upper="1.57" effort="200.0" velocity="4.0"/>
+    <limit lower="0" upper="1" effort="200.0" velocity="4.0"/>
     <dynamics friction="0.0" />
     <axis xyz="0 0 1"/>
@@ -231,5 +231,5 @@
     <child link="leg3_2"/>
     <origin xyz="0.3 0 0"/>
-    <limit lower="-1.57" upper="1.57" effort="200.0" velocity="4"/>
+    <limit lower="0" upper="1" effort="200.0" velocity="4"/>
     <dynamics friction="0.0" />
     <axis xyz="0 0 -1"/>
